File: headphone-audio-amp/headphone-audio-amp.kicad_sch (KiCad schematic)
At the start: 30 parts, among them J1 STEREO OUTPUT, J2 LEFT OUTPUT, J3 RIGHT OUTPUT, U1 NE5532, U2 NE5532

Commit message: General update; also terminates headphone amp's unused opamps
Parts:
- added R1, R2, R3, R4: 10K, symbol Device:R_US
- added unit 2 of U1
- added unit 2 of U2
Connections:
- net +12V: now also R1.1, R3.1
- net GNDPWR: now also R2.2, R4.2
- new net: R3.2, R4.1, U2.5 (+)
- new net: R1.2, R2.1, U1.5 (+)
- new net: U1.6 (-), U1.7
- new net: U2.6 (-), U2.7
Other:
- moved on the sheet: CD1, CD2, CD3, CD4, CD5, CD6, CD7, CD8, RE1, RE10, RE11, RE12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
